File: components/led-matrix/sensors.kicad_sch (KiCad schematic)
At the start: 7 parts, among them U2 CY8CMBR3110, U4 ADAU1361, U7 LTR-303ALS-01, U9 SHT40

Commit message: svg
Parts:
- removed U2: CY8CMBR3110, Package_SO:SOIC-16_3.9x9.9mm_P1.27mm, symbol Sensor_Touch:CY8CMBR3110
- added C14, C15, C16, C17: 0.1uF, Capacitor_SMD:C_0402_1005Metric, symbol PCM_SparkFun-Capacitor:0.1uF_0402_16V_10%
- added JP1, JP10, JP11, JP12, JP13, JP14, JP15, JP16, JP17, JP18, JP19, JP2, JP20, JP21, JP22, JP23, JP24, JP25, JP26, JP27, JP28, JP29, JP3, JP30, JP31, JP32, JP4, JP5, JP6, JP7, JP8, JP9: SolderJumper_2_Bridged, Jumper:SolderJumper-2_P1.3mm_Bridged_RoundedPad1.0x1.5mm, symbol Jumper:SolderJumper_2_Bridged
- added U11, U6: CY8CMBR3116, Package_DFN_QFN:QFN-24-1EP_4x4mm_P0.5mm_EP2.6x2.6mm, symbol Sensor_Touch:CY8CMBR3116
- renumbered U7 to AMB_LIGHT, U9 to TEMP
Connections:
- net +3V3: now also C15.1, C16.1, U11.7 (VDD), U6.7 (VDD)
- net GND: now also C14.1, C15.2, C16.2, C17.1, U11.25 (EP), U11.8 (VSS), U6.25 (EP), U6.8 (VSS)
- net SCL1: now also U6.22 (SCL)
- net SDA1: now also U6.21 (SDA)
- new net: JP4.2 (B), U6.4 (CS3)
- new net: JP25.2 (B), U11.17 (CS7)
- new net: JP22.2 (B), U11.20 (CS4)
- new net: C14.2, U11.6 (VCC)
- new net: JP11.2 (B), U6.14 (CS10)
- new net: JP5.2 (B), U6.20 (CS4)
- new net: JP2.2 (B), U6.2 (CS1)
- new net: JP24.2 (B), U11.18 (CS6)
- new net: JP14.2 (B), U6.12 (CS12)
- new net: JP27.2 (B), U11.15 (CS9)
- new net: JP21.2 (B), U11.4 (CS3)
- new net: C17.2, U6.6 (VCC)
- new net: JP28.2 (B), U11.13 (CS11)
- new net: JP18.2 (B), U11.1 (CS0)
- new net: JP31.2 (B), U11.10 (CS14)
- new net: JP30.2 (B), U11.11 (CS13)
- new net: JP29.2 (B), U11.12 (CS12)
- new net: JP12.2 (B), U11.14 (CS10)
- new net: JP26.2 (B), U11.16 (CS8)
- new net: JP23.2 (B), U11.19 (CS5)
- new net: JP19.2 (B), U11.2 (CS1)
- new net: JP20.2 (B), U11.3 (CS2)
- new net: JP32.2 (B), U11.9 (CS15)
- new net: JP17.2 (B), U6.9 (CS15)
- new net: JP13.2 (B), U6.13 (CS11)
- new net: JP6.2 (B), U6.19 (CS5)
- new net: JP1.2 (B), U6.1 (CS0)
- new net: JP16.2 (B), U6.10 (CS14)
- new net: JP15.2 (B), U6.11 (CS13)
- new net: JP10.2 (B), U6.15 (CS9)
- new net: JP9.2 (B), U6.16 (CS8)
- new net: JP8.2 (B), U6.17 (CS7)
- new net: JP7.2 (B), U6.18 (CS6)
- new net: JP3.2 (B), U6.3 (CS2)
- new net SCL2: U11.22 (SCL)
- new net SDA2: U11.21 (SDA)
- new net T_C0: JP12.1 (A)
- new net T_C1: JP28.1 (A)
- new net T_C2: JP29.1 (A)
- new net T_C3: JP30.1 (A)
- new net T_C4: JP31.1 (A)
- new net T_C5: JP32.1 (A)
- new net T_CL: JP26.1 (A)
- new net T_CL0: JP11.1 (A)
- new net T_CL1: JP13.1 (A)
- new net T_CLI0: JP24.1 (A)
- new net T_CLI1: JP25.1 (A)
- new net T_CR: JP27.1 (A)
- new net T_CR0: JP5.1 (A)
- new net T_CR1: JP6.1 (A)
- new net T_CRI0: JP18.1 (A)
- new net T_CRI1: JP19.1 (A)
- new net T_LL0: JP9.1 (A)
- new net T_LL1: JP10.1 (A)
- new net T_LLI0: JP22.1 (A)
- new net T_LLI1: JP23.1 (A)
- new net T_LR0: JP7.1 (A)
- new net T_LR1: JP8.1 (A)
- new net T_LRI0: JP20.1 (A)
- new net T_LRI1: JP21.1 (A)
- new net T_UL0: JP1.1 (A)
- new net T_UL1: JP2.1 (A)
- new net T_ULI0: JP14.1 (A)
- new net T_ULI1: JP15.1 (A)
- new net T_UR0: JP3.1 (A)
- new net T_UR1: JP4.1 (A)
- new net T_URI0: JP16.1 (A)
- new net T_URI1: JP17.1 (A)
Other:
- note added: "Capacitive sensors"
- note added: "Map of capacitive areas"
