File: cyberdecks/tricorder/rasp-pi.kicad_sch (KiCad schematic)
At the start: 1 part, among them U1 ESP32-S3-WROOM-2

Commit message: 'n sacco de robba
Parts:
- removed U1: ESP32-S3-WROOM-2, PCM_SparkFun-RF:ESP32-S3-WROOM-1, symbol RF_Module:ESP32-S3-WROOM-2
- added J1: Raspberry_Pi_2x20_PTH_NoSilk, PCM_SparkFun-Connector:2x20_Shrouded_NoSilk, symbol PCM_SparkFun-Connector:Raspberry_Pi_2x20_PTH_NoSilk
Connections:
- net -3V3: now also J1.1 (3V3), J1.17 (3V3)
- net GND: now also J1.14 (GND), J1.20 (GND), J1.25 (GND), J1.30 (GND), J1.34 (GND), J1.39 (GND), J1.6 (GND), J1.9 (GND)
- new net: J1.2 (5V), J1.4 (5V)
Changed lines of the file:
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@@
 	(paper "A4")
 	(symbol
-		(lib_id "RF_Module:ESP32-S3-WROOM-2")
-		(at 49.53 100.33 0)
-		(unit 1)
-		(body_style 1)
-		(exclude_from_sim no)
-		(in_bom yes)
-		(on_board yes)
-		(in_pos_files yes)
-		(dnp no)
-		(fields_autoplaced yes)
-		(property "Reference" "U1"
-			(at 51.8968 49.53 0)
-			(show_name no)
-			(do_not_autoplace no)
-			(effects
-				(font
-					(size 1.27 1.27)
-				)
-				(justify left)
-			)
-		)
-		(property "Value" "ESP32-S3-WROOM-2"
-			(at 51.8968 52.07 0)
-			(show_name no)
-			(do_not_autoplace no)
-			(effects
-				(font
-					(size 1.27 1.27)
-				)
-				(justify left)
-			)
-		)
-		(property "Footprint" "PCM_SparkFun-RF:ESP32-S3-WROOM-1"
-			(at 49.53 161.29 0)
-			(hide yes)
-			(show_name no)
-			(do_not_autoplace no)
-			(effects
-				(font
-					(size 1.27 1.27)
-				)
-			)
-		)
-		(property "Datasheet" "https://www.espressif.com/sites/default/files/documentation/esp32-s3-wroom-2_datasheet_en.pdf"
-			(at 49.53 163.83 0)
-			(hide yes)
-			(show_name no)
-			(do_not_autoplace no)
-			(effects
-				(font
-					(size 1.27 1.27)
-				)
-			)
-		)
-		(property "Description" "RF Module, 2.4 GHz, Wi­-Fi, Bluetooth, BLE, ESP32­-S3R8V"
-			(at 49.53 100.33 0)
-			(hide yes)
-			(show_name no)
-			(do_not_autoplace no)
-			(effects
-				(font
-					(size 1.27 1.27)
-				)
-			)
-		)
-		(pin "17"
-		)
-		(pin "24"
-		)
-		(pin "8"
-		)
-		(pin "15"
-		)
-		(pin "9"
-		)
-		(pin "14"
-		)
-		(pin "13"
-		)
-		(pin "12"
-		)
-		(pin "28"
-		)
-		(pin "10"
-		)
-		(pin "20"
-		)
-		(pin "23"
-		)
-		(pin "11"
-		)
-		(pin "18"
-		)
-		(pin "25"
-		)
-		(pin "16"
-		)
-		(pin "26"
-		)
-		(pin "27"
-		)
-		(pin "34"
-		)
-		(pin "35"
-		)
-		(pin "36"
-		)
-		(pin "37"
-		)
-		(pin "29"
-		)
-		(pin "39"
-		)
-		(pin "30"
-		)
-		(pin "31"
-		)
-		(pin "38"
-		)
-		(pin "19"
-		)
-		(pin "1"
-		)
-		(pin "41"
-		)
-		(pin "22"
-		)
-		(pin "33"
-		)
-		(pin "21"
-		)
-		(pin "7"
-		)
-		(pin "6"
-		)
-		(pin "5"
-		)
-		(pin "4"
-		)
-		(pin "3"
-		)
-		(pin "2"
-		)
-		(pin "40"
-		)
-		(pin "32"
-		)
-		(instances
-			(project "tricorder"
-				(path "/6c0a5ebf-5219-47c3-a1b9-62b4178b6e16/484916ad-1214-4f3b-8b2a-9ae7e876ba8f"
-					(reference "U1")
-					(unit 1)
-				)
-			)
-		)
-	)
-	(symbol
 		(lib_id "power:GND")
-		(at 49.53 148.59 0)
+		(at 50.8 116.84 0)
 		(unit 1)
 		(body_style 1)
@@
 		(fields_autoplaced yes)
 		(property "Reference" "#PWR01"
-			(at 49.53 154.94 0)
+			(at 50.8 123.19 0)
 			(hide yes)
 			(show_name no)
@@
 		)
 		(property "Value" "GND"
-			(at 49.53 153.67 0)
+			(at 50.8 121.92 0)
 			(show_name no)
 			(do_not_autoplace no)
@@
 		)
 		(property "Footprint" ""
-			(at 49.53 148.59 0)
+			(at 50.8 116.84 0)
 			(hide yes)
 			(show_name no)
@@
 		)
 		(property "Datasheet" ""
-			(at 49.53 148.59 0)
+			(at 50.8 116.84 0)
 			(hide yes)
 			(show_name no)
@@
 		)
 		(property "Description" "Power symbol creates a global label with name \"GND\" , ground"
-			(at 49.53 148.59 0)
+			(at 50.8 116.84 0)
 			(hide yes)
 			(show_name no)
@@
 	(symbol
 		(lib_id "power:-3V3")
-		(at 49.53 52.07 0)
+		(at 53.34 66.04 0)
 		(unit 1)
 		(body_style 1)
@@
 		(fields_autoplaced yes)
 		(property "Reference" "#PWR02"
-			(at 49.53 55.88 0)
+			(at 53.34 69.85 0)
 			(hide yes)
 			(show_name no)
@@
 		)
 		(property "Value" "-3V3"
-			(at 49.53 46.99 0)
+			(at 53.34 60.96 0)
 			(show_name no)
 			(do_not_autoplace no)
@@
 		)
 		(property "Footprint" ""
-			(at 49.53 52.07 0)
+			(at 53.34 66.04 0)
 			(hide yes)
 			(show_name no)
@@
 		)
 		(property "Datasheet" ""
-			(at 49.53 52.07 0)
+			(at 53.34 66.04 0)
 			(hide yes)
 			(show_name no)
@@
 		)
 		(property "Description" "Power symbol creates a global label with name \"-3V3\""
-			(at 49.53 52.07 0)
+			(at 53.34 66.04 0)
 			(hide yes)
 			(show_name no)
@@
 					(unit 1)
 				)
+			)
+		)
+	)
+	(symbol
+		(lib_id "PCM_SparkFun-Connector:Raspberry_Pi_2x20_PTH_NoSilk")
+		(at 50.8 92.71 0)
+		(unit 1)
+		(body_style 1)
+		(exclude_from_sim no)
+		(in_bom yes)
+		(on_board yes)
+		(in_pos_files yes)
+		(dnp no)
+		(fields_autoplaced yes)
+		(property "Reference" "J1"
+			(at 53.1668 116.84 0)
+			(show_name no)
+			(do_not_autoplace no)
+			(effects
+				(font
+					(size 1.27 1.27)
+				)
+				(justify left)
+			)
+		)
+		(property "Value" "Raspberry_Pi_2x20_PTH_NoSilk"
+			(at 53.1668 119.38 0)
+			(show_name no)
+			(do_not_autoplace no)
+			(effects
+				(font
+					(size 1.27 1.27)
+				)
+				(justify left)
+			)
+		)
+		(property "Footprint" "PCM_SparkFun-Connector:2x20_Shrouded_NoSilk"
+			(at 50.8 137.16 0)
+			(hide yes)
+			(show_name no)
+			(do_not_autoplace no)
+			(effects
+				(font
+					(size 1.27 1.27)
+				)
+			)
+		)
+		(property "Datasheet" "https://www.raspberrypi.org/documentation/hardware/raspberrypi/schematics/rpi_SCH_3bplus_1p0_reduced.pdf"
+			(at 50.8 128.27 0)
+			(hide yes)
+			(show_name no)
+			(do_not_autoplace no)
+			(effects
+				(font
+					(size 1.27 1.27)
+				)
+			)
+		)
+		(property "Description" "SparkFun header for Raspberry Pi"
+			(at 50.8 130.81 0)
+			(hide yes)
+			(show_name no)
+			(do_not_autoplace no)
+			(effects
+				(font
+					(size 1.27 1.27)
+				)
+			)
+		)
+		(property "PROD_ID" "CONN-12263"
+			(at 50.8 133.35 0)
+			(hide yes)
+			(show_name no)
+			(do_not_autoplace no)
+			(effects
+				(font
+					(size 1.27 1.27)
+				)
+			)
+		)
+		(property "SF_ID" "PRT-13054"
+			(at 50.8 135.89 0)
+			(hide yes)
+			(show_name no)
+			(do_not_autoplace no)
+			(effects
+				(font
+					(size 1.27 1.27)
+				)
+			)
+		)
+		(pin "6"
+		)
+		(pin "15"
+		)
+		(pin "14"
+		)
+		(pin "5"
+		)
+		(pin "8"
+		)
+		(pin "13"
+		)
+		(pin "36"
+		)
+		(pin "35"
+		)
+		(pin "24"
+		)
+		(pin "10"
+		)
+		(pin "7"
+		)
+		(pin "33"
+		)
+		(pin "9"
+		)
+		(pin "34"
+		)
+		(pin "16"
+		)
+		(pin "12"
+		)
+		(pin "31"
+		)
+		(pin "23"
+		)
+		(pin "37"
+		)
+		(pin "11"
+		)
+		(pin "17"
+		)
+		(pin "20"
+		)
+		(pin "40"
+		)
+		(pin "22"
+		)
+		(pin "21"
+		)
+		(pin "38"
+		)
+		(pin "32"
+		)
+		(pin "28"
+		)
+		(pin "25"
+		)
+		(pin "19"
+		)
+		(pin "26"
+		)
+		(pin "29"
+		)
+		(pin "27"
+		)
+		(pin "39"
+		)
+		(pin "18"
+		)
+		(pin "1"
+		)
+		(pin "30"
+		)
+		(pin "3"
+		)
+		(pin "2"
+		)
+		(pin "4"
+		)
+		(instances
+			(project "tricorder"
+				(path "/6c0a5ebf-5219-47c3-a1b9-62b4178b6e16/484916ad-1214-4f3b-8b2a-9ae7e876ba8f"
+					(reference "J1")
+					(unit 1)
+				)
