File: cyberdecks/tricorder/tricorder.kicad_sch (KiCad schematic)
At the start: 0 parts

Commit message: 'n sacco de robba
Other:
- sheet MCU renamed R-Pi-Zero-2W
- sheet Untitled Sheet 2 renamed Power source-sink
- added sheet Power sink-only (power-sink-only.kicad_sch)
- sheet Power source-sink: file untitled2.kicad_sch -> power-source-sink.kicad_sch
- sheet R-Pi-Zero-2W: file untitled.kicad_sch -> rasp-pi.kicad_sch
Changed lines of the file:
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@@
 			(color 0 0 0 0)
 		)
-		(property "Sheetname" "MCU"
+		(property "Sheetname" "R-Pi-Zero-2W"
 			(at 25.4 39.9284 0)
 			(show_name no)
@@
 			)
 		)
-		(property "Sheetfile" "untitled.kicad_sch"
+		(property "Sheetfile" "rasp-pi.kicad_sch"
 			(at 25.4 90.7546 0)
 			(show_name no)
@@
 	)
 	(sheet
+		(at 88.9 137.16)
+		(size 43.18 29.21)
+		(exclude_from_sim no)
+		(in_bom yes)
+		(on_board yes)
+		(dnp no)
+		(fields_autoplaced yes)
+		(stroke
+			(width 0.1524)
+			(type solid)
+		)
+		(fill
+			(color 0 0 0 0)
+		)
+		(property "Sheetname" "Power sink-only"
+			(at 88.9 136.4484 0)
+			(show_name no)
+			(do_not_autoplace no)
+			(effects
+				(font
+					(size 1.27 1.27)
+				)
+				(justify left bottom)
+			)
+		)
+		(property "Sheetfile" "power-sink-only.kicad_sch"
+			(at 88.9 166.9546 0)
+			(show_name no)
+			(do_not_autoplace no)
+			(effects
+				(font
+					(size 1.27 1.27)
+				)
+				(justify left top)
+			)
+		)
+		(instances
+			(project "tricorder"
+				(path "/6c0a5ebf-5219-47c3-a1b9-62b4178b6e16"
+					(page "4")
+				)
+			)
+		)
+	)
+	(sheet
 		(at 92.71 31.75)
 		(size 72.39 67.31)
@@
 			(color 0 0 0 0)
 		)
-		(property "Sheetname" "Untitled Sheet 2"
+		(property "Sheetname" "Power source-sink"
 			(at 92.71 31.0384 0)
 			(show_name no)
@@
 			)
 		)
-		(property "Sheetfile" "untitled2.kicad_sch"
+		(property "Sheetfile" "power-source-sink.kicad_sch"
 			(at 92.71 99.6446 0)
 			(show_name no)
