File: lapel/strobo/strobo.kicad_pcb (KiCad board)
At the start: 2 copper layers, 51 x 51 mm, 34 parts, among them J1 USB_C_Receptacle_PowerOnly_6P, SW1 SW_SPDT, U1 ICM7556, U2 MCP73831-2-MC

Commit message: 'n sacco de robba
Parts:
- removed the REF** at (50.0, 28.0)
- removed U1: ICM7556, Package_SO:SOIC-14_3.9x8.7mm_P1.27mm
- added ?: GND, TestPoint:TestPoint_Pad_1.5x1.5mm, F.Cu at (53.8, 66.0)
- added ?: BAT+, TestPoint:TestPoint_Pad_1.5x1.5mm, F.Cu at (64.8, 54.0)
- added ?: GND, TestPoint:TestPoint_Pad_1.5x1.5mm, F.Cu at (44.4, 62.1)
- added ?: GND, TestPoint:TestPoint_Pad_1.5x1.5mm, F.Cu at (61.0, 54.0)
- added ?: 3v3, TestPoint:TestPoint_Pad_1.5x1.5mm, F.Cu at (58.5, 66.0)
- added ?: 5v, TestPoint:TestPoint_Pad_1.5x1.5mm, F.Cu at (47.3, 62.1)
- added B_{1}: 0Ω, Resistor_SMD:R_0603_1608Metric, F.Cu at (52.5, 63.3)
- added REF**: MountingHole_3mm, MountingHole:MountingHole_3mm, F.Cu at (50.0, 28.0)
- added U3: LMC555xTP, Package_BGA:Texas_DSBGA-8_1.43x1.41mm_Layout3x3_P0.5mm, F.Cu at (40.0, 58.0)
- added U4: LMC555xTP, Package_BGA:Texas_DSBGA-8_1.43x1.41mm_Layout3x3_P0.5mm, F.Cu at (58.5, 58.0)
- BT1: value LIR2032 -> 3.7
- C1: footprint Capacitor_SMD:C_0805_2012Metric -> Resistor_SMD:R_0402_1005Metric_Pad0.72x0.64mm_HandSolder
- C2: footprint Capacitor_SMD:C_0805_2012Metric -> Capacitor_SMD:C_0603_1608Metric_Pad1.08x0.95mm_HandSolder
- C3, C4, C5, C6: footprint Capacitor_SMD:C_0805_2012Metric_Pad1.18x1.45mm_HandSolder -> Resistor_SMD:R_0603_1608Metric
- J1: value USB_C_Receptacle_PowerOnly_6P -> USB-C; footprint Connector_USB:USB_C_Receptacle_GCT_USB4125-xx-x-0190_6P_TopMnt_Horizontal -> Connector_USB:USB_C_Receptacle_GCT_USB4135-GF-A_6P_TopMnt_Horizontal
- R1: footprint Resistor_SMD:R_0805_2012Metric_Pad1.20x1.40mm_HandSolder -> Resistor_SMD:R_0402_1005Metric_Pad0.72x0.64mm_HandSolder
- R10, R11, R12, R13, R14, R5, R6, R7, R8, R9: footprint Resistor_SMD:R_0805_2012Metric_Pad1.20x1.40mm_HandSolder -> Resistor_SMD:R_0603_1608Metric
- R2, R3: footprint Capacitor_SMD:C_0805_2012Metric_Pad1.18x1.45mm_HandSolder -> Resistor_SMD:R_0402_1005Metric_Pad0.72x0.64mm_HandSolder
- R4: value 1kΩ -> 470Ω; footprint Resistor_SMD:R_0805_2012Metric_Pad1.20x1.40mm_HandSolder -> Resistor_SMD:R_0603_1608Metric
- SW1: value SW_SPDT -> 0.001; footprint Button_Switch_THT:SW_Slide_SPDT_Angled_CK_OS102011MA1Q -> Button_Switch_SMD:SW_SPST_REED_CT05-XXXX-G1
- moved C5 23.0 mm to (61.0, 57.2), turned to 90 degrees
- moved R7 18.6 mm to (57.7, 55.5), turned to 180 degrees
- moved C6 12.8 mm to (56.8, 60.5), turned to 0 degrees
- moved R8 11.9 mm to (56.0, 57.8), turned to -90 degrees
- moved C3 11.7 mm to (42.5, 57.2), turned to 90 degrees
- moved R5 11.5 mm to (39.2, 55.5)
- moved R2 9.14 mm to (49.5, 66.4), turned to 90 degrees
- moved D1 7.61 mm to (48.1, 65.9), turned to -90 degrees
- moved R4 7.53 mm to (49.7, 63.8), turned to 90 degrees
- moved R6 6.79 mm to (37.5, 57.8), turned to -90 degrees
- moved R1 6.21 mm to (50.5, 66.4), turned to 90 degrees
- moved C4 5.25 mm to (38.4, 60.5), turned to 0 degrees
- moved R3 2.84 mm to (51.6, 61.4), turned to 90 degrees
- moved U2 2.25 mm to (50.0, 58.5)
- moved C1 2.05 mm to (51.5, 66.4), turned to -90 degrees
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Connections:
- C1 pad 1: Net-(C1-Pad1) -> GND
- C1 pad 2: GND -> Net-(D1-A)
- C3 pad 1: Net-(U1A-THRES) -> Net-(U3-TRIG)
- C5 pad 1: Net-(U1B-THRES) -> Net-(U4-TRIG)
- D1 pad 1: GND -> Net-(D1-K)
- J1 pad A9: Net-(C1-Pad1) -> Net-(D1-A)
- J1 pad B9: Net-(C1-Pad1) -> Net-(D1-A)
- R3 pad 1: Net-(U2-PROG) -> GND
- R3 pad 2: GND -> Net-(U2-PROG)
- R4 pad 1: Net-(U2-STAT) -> Net-(D1-K)
- R4 pad 2: Net-(D1-A) -> Net-(U2-STAT)
- R6 pad 2: Net-(U1A-THRES) -> Net-(U3-THRES)
- R8 pad 2: Net-(U1B-THRES) -> Net-(U4-THRES)
- SW1 pad 1: unconnected-(SW1-A-Pad1) -> Net-(BT1-+)
- SW1 pad 2: Net-(BT1-+) -> +3.3V
- U2 pad 1: Net-(C1-Pad1) -> Net-(D1-A)
- U2 pad 2: Net-(C1-Pad1) -> Net-(D1-A)
Routing:
- net Net-(BT1-+): track 65.0 -> 111.9 mm, vias 4 -> 0
- net Net-(D1-A): track 2.00 -> 26.5 mm
- net Net-(U1B-THRES): track 19.3 -> 0.00 mm
- net Net-(C1-Pad1): track 18.6 -> 0.00 mm, vias 2 -> 0
- net Net-(U1A-THRES): track 13.9 -> 0.00 mm
- net Net-(J1-CC1): track 13.8 -> 1.97 mm
- net Net-(D2-A): track 1.79 -> 13.4 mm
- net Net-(D2-K): track 121.2 -> 110.9 mm
- net GND: track 121.0 -> 130.7 mm, vias 2 -> 0
- net Net-(J1-CC2): track 9.55 -> 1.97 mm
- net Net-(U3-CONT): track 9.47 -> 2.11 mm, vias 2 -> 0
- net Net-(D3-K): track 120.8 -> 126.8 mm, vias 6 -> 9
- net Net-(U4-CONT): track 7.12 -> 2.14 mm, vias 2 -> 0
- net Net-(U4-DISCH): track 8.72 -> 4.37 mm
- net Net-(U2-STAT): track 7.62 -> 3.30 mm
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Other:
- board text added: "Designed in Italy"
- board text added: ""
- board text added: "󰊟"
- board text added: "󰢄"
- board text added: "󰢜"
