File: lapel/strobo/strobo.kicad_sch (KiCad schematic)
At the start: 32 parts, among them J1 USB_C_Receptacle_PowerOnly_6P, SW1 0.001, U1 ICM7556, U2 MCP73831-2-MC

Commit message: 'n sacco de robba
Parts:
- removed U1: ICM7556, Package_SO:SOIC-14_3.9x8.7mm_P1.27mm, symbol Timer:ICM7556
- added U3, U4: LMC555xTP, Package_BGA:Texas_DSBGA-8_1.43x1.41mm_Layout3x3_P0.5mm, symbol Timer:LMC555xTP
Connections:
- net +3.3V: now also SW1.1 (A), U3.A2 (VCC), U3.C2 (~{RST}), U4.A2 (VCC), U4.C2 (~{RST}); no longer SW1.3 (C)
- net GND: now also C1.1, R3.1, U3.A3 (GND), U4.A3 (GND); no longer C1.2, D1.1 (K), R3.2
- net at J1.A9 (VBUS), J1.B9 (VBUS), U2.1 (V_{DD})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: now also C1.2, D1.2 (A); no longer C1.1
- net at R5.2, R6.1: now also U3.A1 (DISCH)
- net at R6.2: now also U3.B1 (THRES); no longer C3.1
- net at D3.1 (K), D6.1 (K), D7.1 (K)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: now also U3.C3 (OUT)
- net at R7.2, R8.1: now also U4.A1 (DISCH)
- net at R8.2: now also U4.B1 (THRES); no longer C5.1
- net at C4.2: now also U3.C1 (CONT)
- net at R4.2: now also U2.5 (STAT); no longer D1.2 (A)
- net at U2.8 (PROG): now also R3.2; no longer R3.1
- net at D2.1 (K), D4.1 (K), D5.1 (K)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: now also U4.C3 (OUT)
- net at R4.1: now also D1.1 (K); no longer U2.5 (STAT)
- net at C6.2: now also U4.C1 (CONT)
- new net: C3.1, U3.B3 (TRIG)
- new net: C5.1, U4.B3 (TRIG)
- no-connect marks 0 -> 1
Other:
- moved on the sheet: R3
